File: hardware/radio/controller.sch (KiCad schematic (older format))
At the start: 12 parts, among them IC301 ATMEGA328-A, Q301 Q_NMOS_DGS, X301 8MHz

Commit message: Assign testpoint footprints
Parts:
- C301, C302, C303, C304, C305, C306: footprint (none) -> Capacitors_SMD:C_0603
- D301: footprint (none) -> LEDs:LED-0603
- IC301: footprint TQFP32 -> (none)
- R301, R302: footprint (none) -> Resistors_SMD:R_0603
- X301: footprint (none) -> Crystals_Oscillators_SMD:crystal_FA238-TSX3225
Changed lines of the file:
@@
 F 0 "X301" H 7300 2690 50  0000 C CNN
 F 1 "8MHz" H 7330 2490 50  0000 L CNN
-F 2 "" H 7300 2600 60  0000 C CNN
+F 2 "Crystals_Oscillators_SMD:crystal_FA238-TSX3225" H 7300 2600 60  0001 C CNN
 F 3 "" H 7300 2600 60  0000 C CNN
 	1    7300 2600
@@
 F 0 "C304" H 7625 3100 50  0000 L CNN
 F 1 "22p" H 7625 2900 50  0000 L CNN
-F 2 "" H 7638 2850 30  0000 C CNN
+F 2 "Capacitors_SMD:C_0603" H 7638 2850 30  0001 C CNN
 F 3 "" H 7600 3000 60  0000 C CNN
 	1    7600 3000
@@
 F 0 "C303" H 7025 3100 50  0000 L CNN
 F 1 "22p" H 7025 2900 50  0000 L CNN
-F 2 "" H 7038 2850 30  0000 C CNN
+F 2 "Capacitors_SMD:C_0603" H 7038 2850 30  0001 C CNN
 F 3 "" H 7000 3000 60  0000 C CNN
 	1    7000 3000
@@
 $EndComp
 $Comp
-L GND #PWR028
+L GND #PWR029
 U 1 1 55EA8C66
 P 7600 3250
-F 0 "#PWR028" H 7600 3000 50  0001 C CNN
+F 0 "#PWR029" H 7600 3000 50  0001 C CNN
 F 1 "GND" H 7600 3100 50  0000 C CNN
 F 2 "" H 7600 3250 60  0000 C CNN
@@
 $EndComp
 $Comp
-L GND #PWR029
+L GND #PWR030
 U 1 1 55EA8C82
 P 7300 3250
-F 0 "#PWR029" H 7300 3000 50  0001 C CNN
+F 0 "#PWR030" H 7300 3000 50  0001 C CNN
 F 1 "GND" H 7300 3100 50  0000 C CNN
 F 2 "" H 7300 3250 60  0000 C CNN
@@
 $EndComp
 $Comp
-L GND #PWR030
+L GND #PWR031
 U 1 1 55EA8C9E
 P 7000 3250
-F 0 "#PWR030" H 7000 3000 50  0001 C CNN
+F 0 "#PWR031" H 7000 3000 50  0001 C CNN
 F 1 "GND" H 7000 3100 50  0000 C CNN
 F 2 "" H 7000 3250 60  0000 C CNN
@@
 F 0 "R301" V 6530 3250 50  0000 C CNN
 F 1 "10k" V 6450 3250 50  0000 C CNN
-F 2 "" V 6380 3250 30  0000 C CNN
+F 2 "Resistors_SMD:R_0603" V 6380 3250 30  0001 C CNN
 F 3 "" H 6450 3250 30  0000 C CNN
 	1    6450 3250
@@
 F 0 "C305" H 6475 3750 50  0000 L CNN
 F 1 "100n" H 6475 3550 50  0000 L CNN
-F 2 "" H 6488 3500 30  0000 C CNN
+F 2 "Capacitors_SMD:C_0603" H 6488 3500 30  0001 C CNN
 F 3 "" H 6450 3650 60  0000 C CNN
 	1    6450 3650
@@
 $EndComp
 $Comp
-L VCC #PWR031
+L VCC #PWR032
 U 1 1 55EA9129
 P 6450 3050
-F 0 "#PWR031" H 6450 2900 50  0001 C CNN
+F 0 "#PWR032" H 6450 2900 50  0001 C CNN
 F 1 "VCC" H 6450 3200 50  0000 C CNN
 F 2 "" H 6450 3050 60  0000 C CNN
@@
 $EndComp
 $Comp
-L GND #PWR032
+L GND #PWR033
 U 1 1 55EA91E9
 P 6450 3850
-F 0 "#PWR032" H 6450 3600 50  0001 C CNN
+F 0 "#PWR033" H 6450 3600 50  0001 C CNN
 F 1 "GND" H 6450 3700 50  0000 C CNN
 F 2 "" H 6450 3850 60  0000 C CNN
@@
 TX
 $Comp
-L GND #PWR033
+L GND #PWR034
 U 1 1 55EA9D7E
 P 3200 4750
-F 0 "#PWR033" H 3200 4500 50  0001 C CNN
+F 0 "#PWR034" H 3200 4500 50  0001 C CNN
 F 1 "GND" H 3200 4600 50  0000 C CNN
 F 2 "" H 3200 4750 60  0000 C CNN
@@
 F 0 "C302" H 3225 3050 50  0000 L CNN
 F 1 "100n" H 3225 2850 50  0000 L CNN
-F 2 "" H 3238 2800 30  0000 C CNN
+F 2 "Capacitors_SMD:C_0603" H 3238 2800 30  0001 C CNN
 F 3 "" H 3200 2950 60  0000 C CNN
 	1    3200 2950
@@
 $EndComp
 $Comp
-L GND #PWR034
+L GND #PWR035
 U 1 1 55EA9F10
 P 3200 3250
-F 0 "#PWR034" H 3200 3000 50  0001 C CNN
+F 0 "#PWR035" H 3200 3000 50  0001 C CNN
 F 1 "GND" H 3200 3100 50  0000 C CNN
 F 2 "" H 3200 3250 60  0000 C CNN
@@
 $EndComp
 $Comp
-L VCC #PWR035
+L VCC #PWR036
 U 1 1 55EAA1EE
 P 2900 1850
-F 0 "#PWR035" H 2900 1700 50  0001 C CNN
+F 0 "#PWR036" H 2900 1700 50  0001 C CNN
 F 1 "VCC" H 2900 2000 50  0000 C CNN
 F 2 "" H 2900 1850 60  0000 C CNN
@@
 F 0 "C301" H 2925 2300 50  0000 L CNN
 F 1 "100n" H 2925 2100 50  0000 L CNN
-F 2 "" H 2938 2050 30  0000 C CNN
+F 2 "Capacitors_SMD:C_0603" H 2938 2050 30  0001 C CNN
 F 3 "" H 2900 2200 60  0000 C CNN
 	1    2900 2200
@@
 $EndComp
 $Comp
-L GND #PWR036
+L GND #PWR037
 U 1 1 55EAA376
 P 2900 2400
-F 0 "#PWR036" H 2900 2150 50  0001 C CNN
+F 0 "#PWR037" H 2900 2150 50  0001 C CNN
 F 1 "GND" H 2900 2250 50  0000 C CNN
 F 2 "" H 2900 2400 60  0000 C CNN
@@
 F 0 "D301" H 5950 4750 50  0000 C CNN
 F 1 "LED" H 5950 4550 50  0000 C CNN
-F 2 "" H 5950 4650 60  0000 C CNN
+F 2 "LEDs:LED-0603" H 5950 4650 60  0001 C CNN
 F 3 "" H 5950 4650 60  0000 C CNN
 	1    5950 4650
@@
 F 0 "R302" V 6030 5100 50  0000 C CNN
 F 1 "R" V 5950 5100 50  0000 C CNN
-F 2 "" V 5880 5100 30  0000 C CNN
+F 2 "Resistors_SMD:R_0603" V 5880 5100 30  0001 C CNN
 F 3 "" H 5950 5100 30  0000 C CNN
 	1    5950 5100
@@
 $EndComp
 $Comp
-L GND #PWR037
+L GND #PWR038
 U 1 1 55EACDAA
 P 5950 5400
-F 0 "#PWR037" H 5950 5150 50  0001 C CNN
+F 0 "#PWR038" H 5950 5150 50  0001 C CNN
 F 1 "GND" H 5950 5250 50  0000 C CNN
 F 2 "" H 5950 5400 60  0000 C CNN
@@
 F 0 "Q301" H 2500 2900 50  0000 R CNN
 F 1 "Q_NMOS_DGS" H 2250 2650 50  0000 R CNN
-F 2 "" H 2400 2950 29  0000 C CNN
+F 2 "" H 2400 2950 29  0001 C CNN
 F 3 "" H 2200 2850 60  0000 C CNN
 	1    2200 2850
@@
 $EndComp
 $Comp
-L GND #PWR038
+L GND #PWR039
 U 1 1 55EAF28A
 P 2300 3200
-F 0 "#PWR038" H 2300 2950 50  0001 C CNN
+F 0 "#PWR039" H 2300 2950 50  0001 C CNN
 F 1 "GND" H 2300 3050 50  0000 C CNN
 F 2 "" H 2300 3200 60  0000 C CNN
@@
 F 0 "IC301" H 3650 4350 40  0000 L BNN
 F 1 "ATMEGA328-A" H 4800 1700 40  0000 L BNN
-F 2 "TQFP32" H 4400 3100 30  0000 C CIN
+F 2 "" H 4400 3100 30  0001 C CIN
 F 3 "" H 4400 3100 60  0000 C CNN
 	1    4400 3100
@@
 F 0 "C306" H 3275 2300 50  0000 L CNN
 F 1 "C" H 3275 2100 50  0000 L CNN
-F 2 "" H 3288 2050 30  0000 C CNN
+F 2 "Capacitors_SMD:C_0603" H 3288 2050 30  0001 C CNN
 F 3 "" H 3250 2200 60  0000 C CNN
 	1    3250 2200
@@
 	3250 2350 3250 2400
 $Comp
-L GND #PWR039
+L GND #PWR040
 U 1 1 55ED2A96
 P 3250 2400
-F 0 "#PWR039" H 3250 2150 50  0001 C CNN
+F 0 "#PWR040" H 3250 2150 50  0001 C CNN
 F 1 "GND" H 3250 2250 50  0000 C CNN
 F 2 "" H 3250 2400 60  0000 C CNN

Commit message: Work on laying out TPs
Connections:
- net VCC: no longer C301.1, C306.1, IC301.18 (AVCC), IC301.4 (VCC), IC301.6 (VCC)
- new net VCC_uc: C301.1, C306.1, IC301.18 (AVCC), IC301.4 (VCC), IC301.6 (VCC)
Changed lines of the file:
@@
 $EndComp
 $Comp
-L GND #PWR029
+L GND #PWR027
 U 1 1 55EA8C66
 P 7600 3250
-F 0 "#PWR029" H 7600 3000 50  0001 C CNN
+F 0 "#PWR027" H 7600 3000 50  0001 C CNN
 F 1 "GND" H 7600 3100 50  0000 C CNN
 F 2 "" H 7600 3250 60  0000 C CNN
@@
 $EndComp
 $Comp
-L GND #PWR030
+L GND #PWR028
 U 1 1 55EA8C82
 P 7300 3250
-F 0 "#PWR030" H 7300 3000 50  0001 C CNN
+F 0 "#PWR028" H 7300 3000 50  0001 C CNN
 F 1 "GND" H 7300 3100 50  0000 C CNN
 F 2 "" H 7300 3250 60  0000 C CNN
@@
 $EndComp
 $Comp
-L GND #PWR031
+L GND #PWR029
 U 1 1 55EA8C9E
 P 7000 3250
-F 0 "#PWR031" H 7000 3000 50  0001 C CNN
+F 0 "#PWR029" H 7000 3000 50  0001 C CNN
 F 1 "GND" H 7000 3100 50  0000 C CNN
 F 2 "" H 7000 3250 60  0000 C CNN
@@
 $EndComp
 $Comp
-L VCC #PWR032
+L VCC #PWR030
 U 1 1 55EA9129
 P 6450 3050
-F 0 "#PWR032" H 6450 2900 50  0001 C CNN
+F 0 "#PWR030" H 6450 2900 50  0001 C CNN
 F 1 "VCC" H 6450 3200 50  0000 C CNN
 F 2 "" H 6450 3050 60  0000 C CNN
@@
 $EndComp
 $Comp
-L GND #PWR033
+L GND #PWR031
 U 1 1 55EA91E9
 P 6450 3850
-F 0 "#PWR033" H 6450 3600 50  0001 C CNN
+F 0 "#PWR031" H 6450 3600 50  0001 C CNN
 F 1 "GND" H 6450 3700 50  0000 C CNN
 F 2 "" H 6450 3850 60  0000 C CNN
@@
 TX
 $Comp
-L GND #PWR034
+L GND #PWR032
 U 1 1 55EA9D7E
 P 3200 4750
-F 0 "#PWR034" H 3200 4500 50  0001 C CNN
+F 0 "#PWR032" H 3200 4500 50  0001 C CNN
 F 1 "GND" H 3200 4600 50  0000 C CNN
 F 2 "" H 3200 4750 60  0000 C CNN
@@
 $EndComp
 $Comp
-L GND #PWR035
+L GND #PWR033
 U 1 1 55EA9F10
 P 3200 3250
-F 0 "#PWR035" H 3200 3000 50  0001 C CNN
+F 0 "#PWR033" H 3200 3000 50  0001 C CNN
 F 1 "GND" H 3200 3100 50  0000 C CNN
 F 2 "" H 3200 3250 60  0000 C CNN
 F 3 "" H 3200 3250 60  0000 C CNN
 	1    3200 3250
-	1    0    0    -1
-$EndComp
-$Comp
-L VCC #PWR036
-U 1 1 55EAA1EE
-P 2900 1850
-F 0 "#PWR036" H 2900 1700 50  0001 C CNN
-F 1 "VCC" H 2900 2000 50  0000 C CNN
-F 2 "" H 2900 1850 60  0000 C CNN
-F 3 "" H 2900 1850 60  0000 C CNN
-	1    2900 1850
 	1    0    0    -1
 $EndComp
@@
 $EndComp
 $Comp
-L GND #PWR037
+L GND #PWR034
 U 1 1 55EAA376
 P 2900 2400
-F 0 "#PWR037" H 2900 2150 50  0001 C CNN
+F 0 "#PWR034" H 2900 2150 50  0001 C CNN
 F 1 "GND" H 2900 2250 50  0000 C CNN
 F 2 "" H 2900 2400 60  0000 C CNN
@@
 GND
 Text HLabel 2550 1950 0    60   Input ~ 0
-VCC
+VCC_uc
 $Comp
 L LED D301
@@
 $EndComp
 $Comp
-L GND #PWR038
+L GND #PWR035
 U 1 1 55EACDAA
 P 5950 5400
-F 0 "#PWR038" H 5950 5150 50  0001 C CNN
+F 0 "#PWR035" H 5950 5150 50  0001 C CNN
 F 1 "GND" H 5950 5250 50  0000 C CNN
 F 2 "" H 5950 5400 60  0000 C CNN
@@
 $EndComp
 $Comp
-L GND #PWR039
+L GND #PWR036
 U 1 1 55EAF28A
 P 2300 3200
-F 0 "#PWR039" H 2300 2950 50  0001 C CNN
+F 0 "#PWR036" H 2300 2950 50  0001 C CNN
 F 1 "GND" H 2300 3050 50  0000 C CNN
 F 2 "" H 2300 3200 60  0000 C CNN
@@
 Wire Wire Line
 	3200 3100 3200 3250
-Wire Wire Line
-	2900 1850 2900 2050
 Connection ~ 2900 2000
 Wire Wire Line
@@
 Wire Wire Line
 	2900 1950 2550 1950
-Connection ~ 2900 1950
 Wire Wire Line
 	3200 4650 2850 4650
@@
 	3250 2350 3250 2400
 $Comp
-L GND #PWR040
+L GND #PWR037
 U 1 1 55ED2A96
 P 3250 2400
-F 0 "#PWR040" H 3250 2150 50  0001 C CNN
+F 0 "#PWR037" H 3250 2150 50  0001 C CNN
 F 1 "GND" H 3250 2250 50  0000 C CNN
 F 2 "" H 3250 2400 60  0000 C CNN
@@
 	1    0    0    -1
 $EndComp
+Wire Wire Line
+	2900 1950 2900 2050
 $EndSCHEMATC

Commit message: Assign Q1 footprint
Parts:
- Q301: footprint (none) -> TO_SOT_Packages_SMD:SOT-23
Changed lines of the file:
@@
 F 0 "Q301" H 2500 2900 50  0000 R CNN
 F 1 "Q_NMOS_DGS" H 2250 2650 50  0000 R CNN
-F 2 "" H 2400 2950 29  0001 C CNN
+F 2 "TO_SOT_Packages_SMD:SOT-23" H 2400 2950 29  0001 C CNN
 F 3 "" H 2200 2850 60  0000 C CNN
 	1    2200 2850

Commit message: Parts placed
Connections:
- net VCC is gone; now on net VCC_uc: R301.1
- net UV3: now also IC301.10 ((PCINT22/OC0A/AIN0)PD6); no longer IC301.27 ((PCINT12/SDA/ADC4)PC4)
- net SCL: now reaches IC301.28 ((PCINT13/SCL/ADC5)PC5)
- new net SDA: IC301.27 ((PCINT12/SDA/ADC4)PC4)
Changed lines of the file:
@@
 $EndComp
 $Comp
-L GND #PWR027
+L GND #PWR026
 U 1 1 55EA8C66
 P 7600 3250
-F 0 "#PWR027" H 7600 3000 50  0001 C CNN
+F 0 "#PWR026" H 7600 3000 50  0001 C CNN
 F 1 "GND" H 7600 3100 50  0000 C CNN
 F 2 "" H 7600 3250 60  0000 C CNN
@@
 $EndComp
 $Comp
-L GND #PWR028
+L GND #PWR027
 U 1 1 55EA8C82
 P 7300 3250
-F 0 "#PWR028" H 7300 3000 50  0001 C CNN
+F 0 "#PWR027" H 7300 3000 50  0001 C CNN
 F 1 "GND" H 7300 3100 50  0000 C CNN
 F 2 "" H 7300 3250 60  0000 C CNN
@@
 $EndComp
 $Comp
-L GND #PWR029
+L GND #PWR028
 U 1 1 55EA8C9E
 P 7000 3250
-F 0 "#PWR029" H 7000 3000 50  0001 C CNN
+F 0 "#PWR028" H 7000 3000 50  0001 C CNN
 F 1 "GND" H 7000 3100 50  0000 C CNN
 F 2 "" H 7000 3250 60  0000 C CNN
@@
 $EndComp
 $Comp
-L VCC #PWR030
-U 1 1 55EA9129
-P 6450 3050
-F 0 "#PWR030" H 6450 2900 50  0001 C CNN
-F 1 "VCC" H 6450 3200 50  0000 C CNN
-F 2 "" H 6450 3050 60  0000 C CNN
-F 3 "" H 6450 3050 60  0000 C CNN
-	1    6450 3050
-	1    0    0    -1
-$EndComp
-$Comp
-L GND #PWR031
+L GND #PWR029
 U 1 1 55EA91E9
 P 6450 3850
-F 0 "#PWR031" H 6450 3600 50  0001 C CNN
+F 0 "#PWR029" H 6450 3600 50  0001 C CNN
 F 1 "GND" H 6450 3700 50  0000 C CNN
 F 2 "" H 6450 3850 60  0000 C CNN
@@
 TX
 $Comp
-L GND #PWR032
+L GND #PWR030
 U 1 1 55EA9D7E
 P 3200 4750
-F 0 "#PWR032" H 3200 4500 50  0001 C CNN
+F 0 "#PWR030" H 3200 4500 50  0001 C CNN
 F 1 "GND" H 3200 4600 50  0000 C CNN
 F 2 "" H 3200 4750 60  0000 C CNN
@@
 $EndComp
 $Comp
-L GND #PWR033
+L GND #PWR031
 U 1 1 55EA9F10
 P 3200 3250
-F 0 "#PWR033" H 3200 3000 50  0001 C CNN
+F 0 "#PWR031" H 3200 3000 50  0001 C CNN
 F 1 "GND" H 3200 3100 50  0000 C CNN
 F 2 "" H 3200 3250 60  0000 C CNN
@@
 $EndComp
 $Comp
-L GND #PWR034
+L GND #PWR032
 U 1 1 55EAA376
 P 2900 2400
-F 0 "#PWR034" H 2900 2150 50  0001 C CNN
+F 0 "#PWR032" H 2900 2150 50  0001 C CNN
 F 1 "GND" H 2900 2250 50  0000 C CNN
 F 2 "" H 2900 2400 60  0000 C CNN
@@
 $EndComp
 $Comp
-L GND #PWR035
+L GND #PWR033
 U 1 1 55EACDAA
 P 5950 5400
-F 0 "#PWR035" H 5950 5150 50  0001 C CNN
+F 0 "#PWR033" H 5950 5150 50  0001 C CNN
 F 1 "GND" H 5950 5250 50  0000 C CNN
 F 2 "" H 5950 5400 60  0000 C CNN
@@
 	5900 3150 6000 3250
 Entry Wire Line
-	5900 3250 6000 3350
+	5900 4200 6000 4300
 Entry Wire Line
 	5900 3900 6000 4000
@@
 $EndComp
 $Comp
-L GND #PWR036
+L GND #PWR034
 U 1 1 55EAF28A
 P 2300 3200
-F 0 "#PWR036" H 2300 2950 50  0001 C CNN
+F 0 "#PWR034" H 2300 2950 50  0001 C CNN
 F 1 "GND" H 2300 3050 50  0000 C CNN
 F 2 "" H 2300 3200 60  0000 C CNN
@@
 	5400 3150 5900 3150
 Wire Wire Line
-	5900 3250 5400 3250
+	5900 4200 5400 4200
 Wire Bus Line
 	6000 3050 6000 4450
@@
 Text Label 5450 3150 0    60   ~ 0
 UV2
-Text Label 5450 3250 0    60   ~ 0
+Text Label 5450 4200 0    60   ~ 0
 UV3
 $Comp
@@
 	3250 2350 3250 2400
 $Comp
-L GND #PWR037
+L GND #PWR035
 U 1 1 55ED2A96
 P 3250 2400
-F 0 "#PWR037" H 3250 2150 50  0001 C CNN
+F 0 "#PWR035" H 3250 2150 50  0001 C CNN
 F 1 "GND" H 3250 2250 50  0000 C CNN
 F 2 "" H 3250 2400 60  0000 C CNN
@@
 Wire Wire Line
 	2900 1950 2900 2050
+Text Label 6450 3050 0    60   ~ 0
+VCC_uc
+Wire Wire Line
+	5400 3250 5900 3250
+Wire Wire Line
+	5400 3350 5900 3350
+Text Label 5450 3250 0    60   ~ 0
+SDA
+Text Label 5450 3350 0    60   ~ 0
+SCL
 $EndSCHEMATC

Commit message: Change inductor footprints to 1210
Parts:
- IC301: footprint (none) -> Housings_QFP:TQFP-32_7x7mm_Pitch0.8mm
Changed lines of the file:
@@
 F 0 "IC301" H 3650 4350 40  0000 L BNN
 F 1 "ATMEGA328-A" H 4800 1700 40  0000 L BNN
-F 2 "" H 4400 3100 30  0001 C CIN
+F 2 "Housings_QFP:TQFP-32_7x7mm_Pitch0.8mm" H 4400 3100 30  0001 C CIN
 F 3 "" H 4400 3100 60  0000 C CNN
 	1    4400 3100

Commit message: Routing finalized
Parts:
- removed Q301: Q_NMOS_DGS, TO_SOT_Packages_SMD:SOT-23, symbol Q_NMOS_DGS
- added Q301: BSH105, symbol Q_NMOS_GSD
Connections:
- net EH_ON: now also Q301.1 (G)
- net GND: now also Q301.2 (S)
- net INT1: now also Q301.3 (D)
- no-connect marks 0 -> 4
Changed lines of the file:
@@
 $EndComp
 $Comp
-L GND #PWR026
+L GND #PWR025
 U 1 1 55EA8C66
 P 7600 3250
-F 0 "#PWR026" H 7600 3000 50  0001 C CNN
+F 0 "#PWR025" H 7600 3000 50  0001 C CNN
 F 1 "GND" H 7600 3100 50  0000 C CNN
 F 2 "" H 7600 3250 60  0000 C CNN
@@
 $EndComp
 $Comp
-L GND #PWR027
+L GND #PWR026
 U 1 1 55EA8C82
 P 7300 3250
-F 0 "#PWR027" H 7300 3000 50  0001 C CNN
+F 0 "#PWR026" H 7300 3000 50  0001 C CNN
 F 1 "GND" H 7300 3100 50  0000 C CNN
 F 2 "" H 7300 3250 60  0000 C CNN
@@
 $EndComp
 $Comp
-L GND #PWR028
+L GND #PWR027
 U 1 1 55EA8C9E
 P 7000 3250
-F 0 "#PWR028" H 7000 3000 50  0001 C CNN
+F 0 "#PWR027" H 7000 3000 50  0001 C CNN
 F 1 "GND" H 7000 3100 50  0000 C CNN
 F 2 "" H 7000 3250 60  0000 C CNN
@@
 $EndComp
 $Comp
-L GND #PWR029
+L GND #PWR028
 U 1 1 55EA91E9
 P 6450 3850
-F 0 "#PWR029" H 6450 3600 50  0001 C CNN
+F 0 "#PWR028" H 6450 3600 50  0001 C CNN
 F 1 "GND" H 6450 3700 50  0000 C CNN
 F 2 "" H 6450 3850 60  0000 C CNN
@@
 TX
 $Comp
-L GND #PWR030
+L GND #PWR029
 U 1 1 55EA9D7E
 P 3200 4750
-F 0 "#PWR030" H 3200 4500 50  0001 C CNN
+F 0 "#PWR029" H 3200 4500 50  0001 C CNN
 F 1 "GND" H 3200 4600 50  0000 C CNN
 F 2 "" H 3200 4750 60  0000 C CNN
@@
 $EndComp
 $Comp
-L GND #PWR031
+L GND #PWR030
 U 1 1 55EA9F10
 P 3200 3250
-F 0 "#PWR031" H 3200 3000 50  0001 C CNN
+F 0 "#PWR030" H 3200 3000 50  0001 C CNN
 F 1 "GND" H 3200 3100 50  0000 C CNN
 F 2 "" H 3200 3250 60  0000 C CNN
@@
 $EndComp
 $Comp
-L GND #PWR032
+L GND #PWR031
 U 1 1 55EAA376
 P 2900 2400
-F 0 "#PWR032" H 2900 2150 50  0001 C CNN
+F 0 "#PWR031" H 2900 2150 50  0001 C CNN
 F 1 "GND" H 2900 2250 50  0000 C CNN
 F 2 "" H 2900 2400 60  0000 C CNN
@@
 $EndComp
 $Comp
-L GND #PWR033
+L GND #PWR032
 U 1 1 55EACDAA
 P 5950 5400
-F 0 "#PWR033" H 5950 5150 50  0001 C CNN
+F 0 "#PWR032" H 5950 5150 50  0001 C CNN
 F 1 "GND" H 5950 5250 50  0000 C CNN
 F 2 "" H 5950 5400 60  0000 C CNN
@@
 EH_ON
 $Comp
-L Q_NMOS_DGS Q301
-U 1 1 55EAF184
-P 2200 2850
-F 0 "Q301" H 2500 2900 50  0000 R CNN
-F 1 "Q_NMOS_DGS" H 2250 2650 50  0000 R CNN
-F 2 "TO_SOT_Packages_SMD:SOT-23" H 2400 2950 29  0001 C CNN
-F 3 "" H 2200 2850 60  0000 C CNN
-	1    2200 2850
-	1    0    0    -1
-$EndComp
-$Comp
-L GND #PWR034
+L GND #PWR033
 U 1 1 55EAF28A
 P 2300 3200
-F 0 "#PWR034" H 2300 2950 50  0001 C CNN
+F 0 "#PWR033" H 2300 2950 50  0001 C CNN
 F 1 "GND" H 2300 3050 50  0000 C CNN
 F 2 "" H 2300 3200 60  0000 C CNN
@@
 	3250 2350 3250 2400
 $Comp
-L GND #PWR035
+L GND #PWR034
 U 1 1 55ED2A96
 P 3250 2400
-F 0 "#PWR035" H 3250 2150 50  0001 C CNN
+F 0 "#PWR034" H 3250 2150 50  0001 C CNN
 F 1 "GND" H 3250 2250 50  0000 C CNN
 F 2 "" H 3250 2400 60  0000 C CNN
@@
 Wire Wire Line
 	5400 3250 5900 3250
-Wire Wire Line
-	5400 3350 5900 3350
 Text Label 5450 3250 0    60   ~ 0
 SDA
 Text Label 5450 3350 0    60   ~ 0
 SCL
+NoConn ~ 5400 2000
+NoConn ~ 3500 3350
+NoConn ~ 3500 3450
+NoConn ~ 5400 4300
+Wire Wire Line
+	5400 3350 5750 3350
+Wire Wire Line
+	5750 3350 5750 3300
+Wire Wire Line
+	5750 3300 5900 3300
+$Comp
+L Q_NMOS_GSD Q301
+U 1 1 55F6F2FC
+P 2200 2850
+F 0 "Q301" H 2500 2900 50  0000 R CNN
+F 1 "BSH105" H 2850 2800 50  0000 R CNN
+F 2 "" H 2400 2950 29  0000 C CNN
+F 3 "" H 2200 2850 60  0000 C CNN
+	1    2200 2850
+	1    0    0    -1
+$EndComp
 $EndSCHEMATC
